File: tps63070-module.sch (KiCad schematic (older format))
At the start: 23 parts, among them J1 Conn_01x02_Male, J2 Conn_01x02_Male, J3 Conn_01x03_Male, J4 Conn_01x01_Male, J5 Conn_01x02_Male, J6 Conn_01x02_Male, U1 tps63070

Commit message: Add 3d models
Parts:
- L1: footprint Inductor_SMD:L_Coilcraft_XxL4020 -> tps63070:L_Coilcraft_XxL4020
Changed lines of the file:
@@
 EESchema Schematic File Version 4
+LIBS:tps63070-module-cache
 EELAYER 29 0
 EELAYER END
@@
 F 0 "L1" V 6090 2650 50  0000 C CNN
 F 1 "L" V 5999 2650 50  0000 C CNN
-F 2 "Inductor_SMD:L_Coilcraft_XxL4020" H 5900 2650 50  0001 C CNN
+F 2 "tps63070:L_Coilcraft_XxL4020" H 5900 2650 50  0001 C CNN
 F 3 "~" H 5900 2650 50  0001 C CNN
 	1    5900 2650
